File: hardware/kicad/esp32_breakout/esp32_breakout.kicad_sch (KiCad schematic)
At the start: 17 parts, among them J1 JST PH 8-pin male, J2 JST XH 5-pin male, J3 Deans T-Plug Male, J4 Barrel_Jack, J5 JST XH 5-pin male, J6 Conn_01x03, J7 Conn_01x03, J8 Conn_01x03, U1 ESP32 DEV KIT DOIT 30-pin, U2 MH-KC24

Commit message: KiCad PCB work-in-progress
Parts:
- removed J1: JST PH 8-pin male, symbol Connector_Generic:Conn_01x08
- removed J3: Deans T-Plug Male, symbol Connector_Generic:Conn_01x02
- removed J6, J7, J8: Conn_01x03, symbol Connector_Generic:Conn_01x03
- added D1: 1N4004, symbol Device:D
- added J1: JST PH 2mm 7-pin male thru vertical, symbol Connector_Generic:Conn_01x07
- added J3, J6, J7: JST PH 6-pin male thru vertical, Connector_JST:JST_PH_B6B-PH-K_1x06_P2.00mm_Vertical, symbol Connector_Generic:Conn_01x06
- added Q1: BSS123, Package_TO_SOT_SMD:SOT-23, symbol Transistor_FET:BSS123
- added R8: 1k, Resistor_SMD:R_0603_1608Metric, symbol Device:R_Small_US
- added R9: 4.7k, Resistor_SMD:R_0603_1608Metric, symbol Device:R_Small_US
- added SW1: SS12D10, symbol Switch:SW_SPST
- J2, J5: value JST XH 5-pin male -> JST PH 5-pin male thru vertical; footprint (none) -> Connector_JST:JST_PH_B5B-PH-K_1x05_P2.00mm_Vertical
- R1, R2, R3, R4, R5, R6, R7: footprint (none) -> Resistor_SMD:R_0603_1608Metric
Connections:
- net +24V: now also SW1.1 (A); no longer J4.1
- net +5V: now also D1.1 (K), J1.1 (Pin_1), J3.1 (Pin_1), J6.1 (Pin_1), J7.1 (Pin_1)
- net GND: now also J1.4 (Pin_4), J3.6 (Pin_6), J6.6 (Pin_6), J7.6 (Pin_6), Q1.3 (D)
- net LDS_MOT_EN: now also J1.7 (Pin_7), R8.2
- net LDS_MOT_PWM: now also J1.5 (Pin_5)
- net LDS_RX: now also J1.3 (Pin_3)
- net LDS_TX: now also J1.2 (Pin_2)
- net +3V3: now reaches U1.1 (3V3)
- net +3V3: now also J3.2 (Pin_2), J6.2 (Pin_2), J7.2 (Pin_2), R9.1
- net I2C_SDA: now reaches U1.11 (GPIO21/I2C_SDA)
- net I2C_SDA: now also J3.4 (Pin_4), J6.4 (Pin_4), J7.4 (Pin_4), R9.2
- net I2C_SCL: now reaches U1.14 (GPIO22/I2C_SCL)
- net I2C_SCL: now also J3.3 (Pin_3), J6.3 (Pin_3), J7.3 (Pin_3)
- net I2C_INT: now reaches U1.18 (RTC_GPIO3/SENSOR_VN/ADC1_CH3/GPIO39_IN)
- net I2C_INT: now also J3.5 (Pin_5), J6.5 (Pin_5), J7.5 (Pin_5)
- net TOUCH9: now reaches U1.21 (RTC_GPIO9/TOUCH9/ADC1_CH4/GPIO32)
- net TOUCH6_TBD: now reaches U1.26 (RTC_GPIO16/HSPI_CLK/TOUCH6/ADC2_CH6/GPIO14_BOOT_PWM)
- net TOUCH5_TBD: now reaches U1.27 (RTC_GPIO15/HSPI_MISO/TOUCH5/ADC2_CH5/GPIO12_OUT)
- net TOUCH0: now reaches U1.5 (GPIO4/ADC2_CH0/TOUCH0/RTC_GPIO10)
- new net: D1.2 (A), J1.6 (Pin_6), Q1.2 (S)
- new net: J4.1, SW1.2 (B)
- new net: Q1.1 (G), R8.1
- no-connect marks 10 -> 5
Other:
- note added: "BATTERY"
- note added: "BATTERY CONNECTOR"
- note added: "EXPANSION"
- note added: "TODO - on/off switch footprint - sonar conn? radar conn? - Try GPIO14_BOOT_PWM TOUCH6 - Try GPIO12_OUT TOUCH5 - regulator module connections - charger? - ESP32 footprint - TOUCH connector?"
- note removed: "BATTERY PACK CONNECTOR"
- note removed: "CHARGER/DOCK"
- title: Maker's Pet Snoopy -> ESP32 Breakout
