Commit message: URDF fix

File: urdf/makerspet_snoopy.urdf.xacro (robot description, xacro)
@@ -1,4 +1,4 @@
 <?xml version="1.0" ?>
-<robot name="kaia_snoopy" xmlns:xacro="http://ros.org/wiki/xacro">
+<robot name="makerspet_snoopy" xmlns:xacro="http://ros.org/wiki/xacro">
   <!-- https://classic.gazebosim.org/tutorials?tut=ros_gzplugins&cat=connect_ros -->
   <!-- https://classic.gazebosim.org/tutorials?tut=ros_urdf&cat=connect_ros -->
@@ -281,5 +281,5 @@
       <origin xyz="0 0 0" rpy="0 0 0"/>
       <geometry>
-        <mesh filename="package://kaia_snoopy_description/sdf/kaia_snoopy/mesh/head.stl" scale="${0.001*base_diameter} ${0.001*base_diameter} ${0.001*head_height*2}"/>
+        <mesh filename="package://makerspet_snoopy/sdf/makerspet_snoopy/mesh/head.stl" scale="${0.001*base_diameter} ${0.001*base_diameter} ${0.001*head_height*2}"/>
       </geometry>
       <material name="red"/>
@@ -502,5 +502,5 @@
       <plugin filename="libgazebo_ros_imu_sensor.so" name="imu_plugin">
         <ros>
-          <!-- namespace>/kaia_snoopy</namespace -->
+          <!-- namespace>/robot_instance_1</namespace -->
           <remapping>~/out:=imu</remapping>
         </ros>

Commit message: SDF fix

File: urdf/makerspet_snoopy.urdf.xacro (robot description, xacro)
@@ -281,5 +281,5 @@
       <origin xyz="0 0 0" rpy="0 0 0"/>
       <geometry>
-        <mesh filename="package://makerspet_snoopy/sdf/makerspet_snoopy/mesh/head.stl" scale="${0.001*base_diameter} ${0.001*base_diameter} ${0.001*head_height*2}"/>
+        <mesh filename="package://makerspet_snoopy/mesh/head.stl" scale="${0.001*base_diameter} ${0.001*base_diameter} ${0.001*head_height*2}"/>
       </geometry>
       <material name="red"/>

Commit message: URDF wheel base fix

File: urdf/makerspet_snoopy.urdf.xacro (robot description, xacro)
@@ -14,5 +14,5 @@
   <xacro:property name="floor_clearance" value="0.018"/>
   <xacro:property name="base_diameter" value="0.300"/>
-  <xacro:property name="wheel_base" value="0.131397"/>
+  <xacro:property name="wheel_base" value="262.794"/>
   <xacro:property name="lower_cylinder_height" value="0.119"/>
   <xacro:property name="lower_to_upper_cylinders_gap" value="0.026"/>

Commit message: URDF base fix

File: urdf/makerspet_snoopy.urdf.xacro (robot description, xacro)
@@ -14,5 +14,5 @@
   <xacro:property name="floor_clearance" value="0.018"/>
   <xacro:property name="base_diameter" value="0.300"/>
-  <xacro:property name="wheel_base" value="262.794"/>
+  <xacro:property name="wheel_base" value="0.262794"/>
   <xacro:property name="lower_cylinder_height" value="0.119"/>
   <xacro:property name="lower_to_upper_cylinders_gap" value="0.026"/>

Commit message: Teleop params cleanup

File: urdf/makerspet_snoopy.urdf.xacro (robot description, xacro)
@@ -189,5 +189,5 @@
     <parent link="base_link"/>
     <child link="wheel_left_link"/>
-    <origin xyz="0 ${wheel_base/2} ${wheel_diameter/2-floor_clearance}" rpy="-${pi/2} 0 0"/>
+    <origin xyz="0 ${wheel_base/2} ${wheel_diameter/2-floor_clearance}" rpy="${pi/2} 0 0"/>
     <axis xyz="0 0 1"/>
   </joint>

Commit message: URDF base_scan fix

File: urdf/makerspet_snoopy.urdf.xacro (robot description, xacro)
@@ -233,5 +233,5 @@
     <parent link="base_link"/>
     <child link="base_scan"/>
-    <origin xyz="0 0 ${lower_cylinder_height + (lower_to_upper_cylinders_gap - laser_puck_to_upper_cylinder_gap)/2}" rpy="0 0 0"/>
+    <origin xyz="0 0 ${lower_cylinder_height + (lower_to_upper_cylinders_gap - laser_puck_to_upper_cylinder_gap)/2}" rpy="-${pi} 0 0"/>
   </joint>
   <link name="base_scan">

Commit message: URDF cmd_vel fix

File: urdf/makerspet_snoopy.urdf.xacro (robot description, xacro)
@@ -189,5 +189,5 @@
     <parent link="base_link"/>
     <child link="wheel_left_link"/>
-    <origin xyz="0 ${wheel_base/2} ${wheel_diameter/2-floor_clearance}" rpy="${pi/2} 0 0"/>
+    <origin xyz="0 ${wheel_base/2} ${wheel_diameter/2-floor_clearance}" rpy="-${pi/2} 0 0"/>
     <axis xyz="0 0 1"/>
   </joint>

Commit message: Battery weight

File: urdf/makerspet_snoopy.urdf.xacro (robot description, xacro)
@@ -39,5 +39,6 @@
   <xacro:property name="max_wheel_acceleration" value="5"/>
   <xacro:property name="lower_cylinder_mass" value="0.500"/>
-  <xacro:property name="caster_mass" value="0.020"/>
+  <!-- caster and battery weight -->
+  <xacro:property name="caster_mass" value="0.120"/>
   <xacro:property name="wheel_mass" value="0.050"/>
   <xacro:property name="laser_puck_mass" value="0.200"/>
