File: kicad/esp32_breakout/esp32_breakout.kicad_sch (KiCad schematic)
At the start: 25 parts, among them J1 JST B5B-PH-K-S, J10 JST B6B-PH-K-S, J2 JST B5B-PH-K-S, J3 JST B7B-PH-K-S, J4 XT30U-M, J5 HDR M VERT 12p 2.54mm, J9 JST B6B-PH-K-S, SW1 SS12D10, U1 ESP32 DEV KIT Module 30-pin, U2 LM2596 Module

Commit message: Neato adapter PCB Gerber
Parts:
- H1, H2, H3, H4: now left out of the parts list
Changed lines of the file:
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@@
   )
   (symbol (lib_id "Mechanical:MountingHole") (at 134.62 173.99 0) (unit 1)
-    (in_bom yes) (on_board yes) (dnp no) (fields_autoplaced)
+    (in_bom no) (on_board yes) (dnp no) (fields_autoplaced)
     (property "Reference" "H1" (at 137.16 172.72 0)
       (effects (font (size 1.27 1.27)) (justify left))
@@
   )
   (symbol (lib_id "Mechanical:MountingHole") (at 134.62 193.04 0) (unit 1)
-    (in_bom yes) (on_board yes) (dnp no) (fields_autoplaced)
+    (in_bom no) (on_board yes) (dnp no) (fields_autoplaced)
     (property "Reference" "H4" (at 137.16 191.77 0)
       (effects (font (size 1.27 1.27)) (justify left))
@@
   )
   (symbol (lib_id "Mechanical:MountingHole") (at 134.5851 186.6785 0) (unit 1)
-    (in_bom yes) (on_board yes) (dnp no) (fields_autoplaced)
+    (in_bom no) (on_board yes) (dnp no) (fields_autoplaced)
     (property "Reference" "H3" (at 137.1251 185.4085 0)
       (effects (font (size 1.27 1.27)) (justify left))
@@
   )
   (symbol (lib_id "Mechanical:MountingHole") (at 134.62 180.34 0) (unit 1)
-    (in_bom yes) (on_board yes) (dnp no) (fields_autoplaced)
+    (in_bom no) (on_board yes) (dnp no) (fields_autoplaced)
     (property "Reference" "H2" (at 137.16 179.07 0)
       (effects (font (size 1.27 1.27)) (justify left))
